File: averell4evse/averell4evse.sch (KiCad schematic (older format))
At the start: 31 parts

Commit message: averell/sch: Annotate schematic
Parts:
- gave numbers to parts that had none: 31

Commit message: averell/sch: Assign PCB footprints
Parts:
- C1, C2: footprint (none) -> Capacitor_SMD:C_0603_1608Metric
- J1: footprint (none) -> Connector_PinHeader_2.54mm:PinHeader_1x16_P2.54mm_Horizontal
- J2: footprint (none) -> Connector_PinHeader_2.54mm:PinHeader_1x12_P2.54mm_Horizontal
- J3: footprint (none) -> Connector_PinHeader_2.54mm:PinHeader_1x04_P2.54mm_Horizontal
- R1: footprint (none) -> Resistor_SMD:R_0603_1608Metric
- TP1, TP10, TP11, TP12, TP2, TP3, TP4, TP5, TP6, TP7, TP8, TP9: footprint (none) -> TestPoint:TestPoint_Pad_1.0x1.0mm
- U4: footprint (none) -> Package_TO_SOT_SMD:SOT-23-5
Changed lines of the file:
@@
 F 0 "R1" H 3942 6696 50  0000 R CNN
 F 1 "8k" H 3942 6605 50  0000 R CNN
-F 2 "" H 4000 6650 50  0001 C CNN
+F 2 "Resistor_SMD:R_0603_1608Metric" H 4000 6650 50  0001 C CNN
 F 3 "~" H 4000 6650 50  0001 C CNN
 	1    4000 6650
@@
 F 0 "C2" V 2671 2950 50  0000 C CNN
 F 1 "1u" V 2762 2950 50  0000 C CNN
-F 2 "" H 2900 2950 50  0001 C CNN
+F 2 "Capacitor_SMD:C_0603_1608Metric" H 2900 2950 50  0001 C CNN
 F 3 "~" H 2900 2950 50  0001 C CNN
 	1    2900 2950
@@
 F 0 "C1" V 4071 1550 50  0000 C CNN
 F 1 "1u" V 4162 1550 50  0000 C CNN
-F 2 "" H 4300 1550 50  0001 C CNN
+F 2 "Capacitor_SMD:C_0603_1608Metric" H 4300 1550 50  0001 C CNN
 F 3 "~" H 4300 1550 50  0001 C CNN
 	1    4300 1550
@@
 F 0 "U4" H 3200 4450 50  0000 C CNN
 F 1 "74AUC1G126" H 3050 4350 50  0000 C CNN
-F 2 "" H 3300 4650 50  0001 C CNN
+F 2 "Package_TO_SOT_SMD:SOT-23-5" H 3300 4650 50  0001 C CNN
 F 3 "http://www.ti.com/lit/sg/scyt129e/scyt129e.pdf" H 3300 4650 50  0001 C CNN
 	1    3300 4650
@@
 F 0 "J2" H 1018 5267 50  0000 C CNN
 F 1 "Conn_01x12" H 1018 5176 50  0000 C CNN
-F 2 "" H 1100 4550 50  0001 C CNN
+F 2 "Connector_PinHeader_2.54mm:PinHeader_1x12_P2.54mm_Horizontal" H 1100 4550 50  0001 C CNN
 F 3 "~" H 1100 4550 50  0001 C CNN
 	1    1100 4550
@@
 F 0 "J1" H 9830 3942 50  0000 L CNN
 F 1 "Conn_01x16" H 9830 3851 50  0000 L CNN
-F 2 "" H 9750 3950 50  0001 C CNN
+F 2 "Connector_PinHeader_2.54mm:PinHeader_1x16_P2.54mm_Horizontal" H 9750 3950 50  0001 C CNN
 F 3 "~" H 9750 3950 50  0001 C CNN
 	1    9750 3950
@@
 F 0 "J3" H 9830 5042 50  0000 L CNN
 F 1 "Conn_01x04" H 9830 4951 50  0000 L CNN
-F 2 "" H 9750 5050 50  0001 C CNN
+F 2 "Connector_PinHeader_2.54mm:PinHeader_1x04_P2.54mm_Horizontal" H 9750 5050 50  0001 C CNN
 F 3 "~" H 9750 5050 50  0001 C CNN
 	1    9750 5050
@@
 F 0 "TP1" V 8250 3950 50  0000 C CNN
 F 1 "AUX1" V 8250 4200 50  0000 C CNN
-F 2 "" H 8450 3700 50  0001 C CNN
+F 2 "TestPoint:TestPoint_Pad_1.0x1.0mm" H 8450 3700 50  0001 C CNN
 F 3 "~" H 8450 3700 50  0001 C CNN
 	1    8250 3700
@@
 F 0 "TP2" V 8250 4050 50  0000 C CNN
 F 1 "AUX2" V 8250 4300 50  0000 C CNN
-F 2 "" H 8450 3800 50  0001 C CNN
+F 2 "TestPoint:TestPoint_Pad_1.0x1.0mm" H 8450 3800 50  0001 C CNN
 F 3 "~" H 8450 3800 50  0001 C CNN
 	1    8250 3800
@@
 F 0 "TP3" V 8250 4150 50  0000 C CNN
 F 1 "DBG_RXD" V 8250 4400 50  0000 C CNN
-F 2 "" H 8450 3900 50  0001 C CNN
+F 2 "TestPoint:TestPoint_Pad_1.0x1.0mm" H 8450 3900 50  0001 C CNN
 F 3 "~" H 8450 3900 50  0001 C CNN
 	1    8250 3900
@@
 F 0 "TP4" V 8250 4250 50  0000 C CNN
 F 1 "DBG_TXD" V 8250 4500 50  0000 C CNN
-F 2 "" H 8450 4000 50  0001 C CNN
+F 2 "TestPoint:TestPoint_Pad_1.0x1.0mm" H 8450 4000 50  0001 C CNN
 F 3 "~" H 8450 4000 50  0001 C CNN
 	1    8250 4000
@@
 F 0 "TP5" V 8250 4350 50  0000 C CNN
 F 1 "INT0" V 8250 4600 50  0000 C CNN
-F 2 "" H 8450 4100 50  0001 C CNN
+F 2 "TestPoint:TestPoint_Pad_1.0x1.0mm" H 8450 4100 50  0001 C CNN
 F 3 "~" H 8450 4100 50  0001 C CNN
 	1    8250 4100
@@
 F 0 "TP6" V 8250 4450 50  0000 C CNN
 F 1 "INT1" V 8250 4700 50  0000 C CNN
-F 2 "" H 8450 4200 50  0001 C CNN
+F 2 "TestPoint:TestPoint_Pad_1.0x1.0mm" H 8450 4200 50  0001 C CNN
 F 3 "~" H 8450 4200 50  0001 C CNN
 	1    8250 4200
@@
 F 0 "TP7" V 8250 4550 50  0000 C CNN
 F 1 "SIGCLK" V 8250 4800 50  0000 C CNN
-F 2 "" H 8450 4300 50  0001 C CNN
+F 2 "TestPoint:TestPoint_Pad_1.0x1.0mm" H 8450 4300 50  0001 C CNN
 F 3 "~" H 8450 4300 50  0001 C CNN
 	1    8250 4300
@@
 F 0 "TP8" V 8250 4650 50  0000 C CNN
 F 1 "SIGOUT" V 8250 4900 50  0000 C CNN
-F 2 "" H 8450 4400 50  0001 C CNN
+F 2 "TestPoint:TestPoint_Pad_1.0x1.0mm" H 8450 4400 50  0001 C CNN
 F 3 "~" H 8450 4400 50  0001 C CNN
 	1    8250 4400
@@
 F 0 "TP9" V 8250 4750 50  0000 C CNN
 F 1 "SIGIN" V 8250 5000 50  0000 C CNN
-F 2 "" H 8450 4500 50  0001 C CNN
+F 2 "TestPoint:TestPoint_Pad_1.0x1.0mm" H 8450 4500 50  0001 C CNN
 F 3 "~" H 8450 4500 50  0001 C CNN
 	1    8250 4500
@@
 F 0 "TP10" V 5300 6300 50  0000 C CNN
 F 1 "R13" V 5300 6550 50  0000 C CNN
-F 2 "" H 5500 6050 50  0001 C CNN
+F 2 "TestPoint:TestPoint_Pad_1.0x1.0mm" H 5500 6050 50  0001 C CNN
 F 3 "~" H 5500 6050 50  0001 C CNN
 	1    5300 6050
@@
 F 0 "TP11" V 5300 6400 50  0000 C CNN
 F 1 "G13" V 5300 6650 50  0000 C CNN
-F 2 "" H 5500 6150 50  0001 C CNN
+F 2 "TestPoint:TestPoint_Pad_1.0x1.0mm" H 5500 6150 50  0001 C CNN
 F 3 "~" H 5500 6150 50  0001 C CNN
 	1    5300 6150
@@
 F 0 "TP12" V 5300 6500 50  0000 C CNN
 F 1 "B13" V 5300 6750 50  0000 C CNN
-F 2 "" H 5500 6250 50  0001 C CNN
+F 2 "TestPoint:TestPoint_Pad_1.0x1.0mm" H 5500 6250 50  0001 C CNN
 F 3 "~" H 5500 6250 50  0001 C CNN
 	1    5300 6250
