File: averell4evse/triled.sch (KiCad schematic (older format))
At the start: 3 parts

Commit message: averell: Replace test pads with 0.1" pin headers
Changed lines of the file:
@@
 EESchema Schematic File Version 4
+LIBS:averell4evse-cache
 EELAYER 29 0
 EELAYER END
@@
 AR Path="/5E36EEF8/5E1B05FE" Ref="D19"  Part="1"
 AR Path="/5E36EEFD/5E1B05FE" Ref="D22"  Part="1"
-F 0 "D1" H 5100 3967 50  0000 C CNN
+F 0 "D22" H 5100 3967 50  0000 C CNN
 F 1 "ASMB-MTB0-0A3A2" H 5100 3876 50  0000 C CNN
 F 2 "ma4evse:LED_Avago_PLCC4_3.2x2.8mm_CW" H 5100 3950 50  0001 C CNN
@@
 AR Path="/5E36EEF8/5E1B063C" Ref="D20"  Part="1"
 AR Path="/5E36EEFD/5E1B063C" Ref="D23"  Part="1"
-F 0 "D2" H 6050 3967 50  0000 C CNN
+F 0 "D23" H 6050 3967 50  0000 C CNN
 F 1 "ASMB-MTB0-0A3A2" H 6050 3876 50  0000 C CNN
 F 2 "ma4evse:LED_Avago_PLCC4_3.2x2.8mm_CW" H 6050 3950 50  0001 C CNN
@@
 AR Path="/5E36EEF8/5E1B0F79" Ref="D21"  Part="1"
 AR Path="/5E36EEFD/5E1B0F79" Ref="D24"  Part="1"
-F 0 "D3" H 7000 3967 50  0000 C CNN
+F 0 "D24" H 7000 3967 50  0000 C CNN
 F 1 "ASMB-MTB0-0A3A2" H 7000 3876 50  0000 C CNN
 F 2 "ma4evse:LED_Avago_PLCC4_3.2x2.8mm_CW" H 7000 3950 50  0001 C CNN
