File: joe4evse/relay.sch (KiCad schematic (older format))
At the start: 40 parts, among them J17 Conn_01x03, J18 Conn_01x03, J19 Conn_01x03, J20 Conn_01x03, J21 Conn_01x03, J22 Conn_01x03, J23 Conn_01x03, J24 Conn_01x03, K10 G5LE-1, K11 G5LE-1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

Commit message: joe/sch: Assign footprints to components
Parts:
- removed D15, D16, D17, D18, D19, D20, D22: D_Schottky, Diode_SMD:D_SOD-123, symbol Device:D_Schottky
- removed J17, J18, J19, J20, J21, J23, J24: Conn_01x03, symbol Connector_Generic:Conn_01x03
- removed K11, K12, K13, K14, K15, K16, K9: G5LE-1, Relay_THT:Relay_SPDT_Omron-G5LE-1, symbol Relay:G5LE-1
- removed Q10, Q11, Q12, Q13, Q14, Q16, Q9: AO3402, Package_TO_SOT_SMD:SOT-23, symbol ma4evse:AO3402
- removed R15, R16, R17, R18, R19, R20, R22: 10k, Resistor_SMD:R_0603_1608Metric, symbol Device:R_Small
- J10: renamed from J22; footprint (none) -> Connector_JST:JST_NV_B03P-NV_1x03_P5.00mm_Vertical
- renumbered D21 to D8, K10 to K2, Q15 to Q2, R21 to R8
Connections:
- wire segments 200 -> 25
