File: joe4evse/fipy.sch (KiCad schematic (older format))
At the start: 19 parts, among them J13 Conn_01x03, J8 Conn_01x02, Q4 AO3401A, Q5 AO3402, U3 FiPy, U4 MCP23S08-SO

Commit message: joe/{sch, pcb}: Remove input shottky diodes
Connections:
- net IO_IRQ: now also U4.8 (INT)
Changed lines of the file:
@@
 Wire Wire Line
 	8800 5050 8800 5150
+Wire Wire Line
+	7800 3150 7800 2650
 $EndSCHEMATC

Commit message: joe/{sch, pcb}: Add 0r resistors in parallel of SW1 for prod boards
Parts:
- U4: Manufacturer (none) -> Microchip; Manufacturer PN (none) -> MCP23S08-SO
Changed lines of the file:
@@
 F 2 "Package_SO:SOIC-18W_7.5x11.6mm_P1.27mm" H 8800 2200 50  0001 C CNN
 F 3 "https://ww1.microchip.com/downloads/en/DeviceDoc/21919e.pdf" H 8800 2200 50  0001 C CNN
+F 4 "Microchip" H 8100 2150 50  0001 C CNN "Manufacturer"
+F 5 "MCP23S08-SO" H 8100 2150 50  0001 C CNN "Manufacturer PN"
 	1    8100 2150
 	1    0    0    -1
