File: billy4evse/billy4evse.kicad_pcb (KiCad board)
At the start: 2 copper layers, 44 x 98 mm, 34 parts, among them J1 Conn_01x02, J2 Screw_Terminal_01x02, J3 Conn_01x12, J4 Conn_01x12, J5 AudioJack3_SwitchTR, J6 AudioJack3_SwitchTR, J7 USB_B_Micro, J8 AudioJack3_SwitchTR, U1 LoPy, U2 CH340C

Commit message: billy{sch, pcb}: DIN-compatible second draft
Parts:
- removed H1, H2, H3, H4: MountingHole, MountingHole:MountingHole_3mm_Pad_Via
- added REF**: BC-53-6 series, ma4evse:BC-53-6, F.Cu at (146.0, 92.0)
- J5, J6, J8: value AudioJack3_SwitchTR -> AudioJack3; footprint ma4evse:PJ-307C -> ma4evse:JIS-C-6560
- moved J3 113.0 mm to (212.0, 83.7)
- moved J4 85.0 mm to (224.0, 83.7)
- moved J1 66.9 mm to (169.4, 68.4), turned to 180 degrees
- moved U1 40.4 mm to (158.0, 88.5)
- moved R8 40.0 mm to (135.2, 117.8), turned to 270 degrees
- moved C1 39.9 mm to (169.1, 73.3)
- moved R7 38.7 mm to (136.7, 117.8), turned to 270 degrees
- moved C2 36.7 mm to (142.5, 122.0)
- moved R1 36.7 mm to (139.0, 121.0)
- moved R2 36.7 mm to (142.5, 118.5)
- moved R3 36.7 mm to (142.5, 120.0)
- moved D2 36.3 mm to (135.2, 114.3), turned to 90 degrees
- moved J5 35.1 mm to (139.3, 130.9)
- moved J6 35.1 mm to (152.3, 130.9)
- moved J8 35.1 mm to (165.3, 130.9)
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Connections:
- J4 pad 6: /CT2_DET -> /P20
- J4 pad 7: /CT1_DET -> /P19
- J4 pad 8: /CT0_DET -> /P18
- J5 pad R: /CT0_DET -> (no net)
- J6 pad R: /CT1_DET -> (no net)
- J8 pad R: /CT2_DET -> (no net)
- U1 pad 18: /CT0_DET -> /CT1
- U1 pad 19: /CT1 -> /CT2
- U1 pad 20: /CT1_DET -> /P18
- U1 pad 21: /CT2 -> /P19
- U1 pad 22: /CT2_DET -> /P20
Routing:
- net /CT1_DET: track 62.2 -> 0.00 mm
- net /CT0_DET: track 61.5 -> 0.00 mm
- net /CT2_DET: track 55.7 -> 0.00 mm
- net /USB2LOPY: track 6.24 -> 51.4 mm
- net /LOPY2USB: track 6.11 -> 49.6 mm
- net +3V3: track 126.8 -> 87.7 mm, vias 3 -> 4
- net /USB_N: track 46.6 -> 16.4 mm
- net /USB_P: track 46.6 -> 16.9 mm
- net Net-(J1-Pad2): track 3.57 -> 22.8 mm
- net /P10: track 15.2 -> 0.00 mm
- net /P9: track 15.2 -> 0.00 mm
- net /P8: track 15.2 -> 0.00 mm
- net /P12: track 15.2 -> 0.00 mm
- net /P11: track 15.2 -> 0.00 mm
- net /P14: track 15.2 -> 0.00 mm
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Other:
- board size 44 x 98 mm -> 49.7 x 86.4 mm
