File: william4evse/william4evse.kicad_pcb (KiCad board)
At the start: 2 copper layers, 32 x 65 mm, 6 parts, among them J1 Boom_Precision_RJ45-B-1x1, U1 RCMB121, U2 74LVC1G32

Commit message: william: Release v1.3
Other:
- board text added: "Dalton EVSE "William" board rev. 1.3 (c) Tuetuopay 2019 - 2020"
- board text removed: "Dalton EVSE "William" board rev. 1.2 (c) Tuetuopay 2019 - 2020"
Changed lines of the file:
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@@
     (effects (font (size 1 1) (thickness 0.15)) (justify left mirror))
   )
-  (gr_text "Dalton EVSE\n\"William\" board rev. 1.2\n(c) Tuetuopay 2019 - 2020" (at 150 92) (layer B.SilkS)
+  (gr_text "Dalton EVSE\n\"William\" board rev. 1.3\n(c) Tuetuopay 2019 - 2020" (at 150 92) (layer B.SilkS)
     (effects (font (size 1 1) (thickness 0.15)) (justify left mirror))
   )
